Commit message: camera,script

File: catkin_ws/src/motoman/motoman_hc10_support/urdf/hc10.xacro (robot description, xacro)
@@ -4,3 +4,5 @@
   <xacro:motoman_hc10 prefix=""/>
   <xacro:include filename="$(find motoman_hc10_support)/urdf/hc10_gazebo.xacro"/>
+  <xacro:include filename="$(find motoman_hc10_support)/urdf/hc10_cam.xacro"/>
+  <xacro:add_cam parent_link="tool0"/>
 </robot>

File: catkin_ws/src/motoman/motoman_hc10_support/urdf/hc10_macro.xacro (robot description, xacro)
@@ -167,5 +167,7 @@
     </link>
     <gazebo reference="${prefix}link_6_t">
-      <material>Gazebo/Blue</material>
+      <material>G<axis xyz="0 0 0" rpy="0 0 0"/>
+            <limit effort="10000" velocity="1000"/>
+            <dynamics damping="1.0" friction="1.0"/>zebo/Blue</material>
       <mu1>0.2</mu1>
       <mu2>0.2</mu2>
